File: USB.kicad_sch (KiCad schematic)
At the start: 13 parts, among them J401 USB_B_Micro, Q401 S8050, Q402 S8050, U401 CH340C, U402 RCLAMP0524P-N

Commit message: Rename and update layout
Parts:
- FB601: renamed from FB401; symbol Device:Ferrite_Bead -> Device:FerriteBead
- renumbered C503 to C601, C403 to C602, C404 to C603, C402 to C604, F401 to F601, J401 to J601, Q401 to Q601, Q402 to Q602, R401 to R601, R402 to R602, U401 to U601, U402 to U602
Changed lines of the file:
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@@
     (effects (font (size 1.27 1.27)) (justify left))
   )
-  (symbol (lib_id "SH-ESP32:USB_B_Micro-Connector") (at 25.4 44.45 0)
-    (in_bom yes) (on_board yes)
-    (property "Reference" "J401" (id 0) (at 26.8478 32.5882 0))
+  (symbol (lib_id "SH-ESP32:USB_B_Micro-Connector") (at 25.4 44.45 0) (unit 1)
+    (in_bom yes) (on_board yes)
+    (property "Reference" "J601" (id 0) (at 26.8478 32.5882 0))
     (property "Value" "USB_B_Micro" (id 1) (at 26.8478 34.8996 0))
     (property "Footprint" "Connector_USB:USB_Micro-B_Wuerth_614105150721_Vertical" (id 2) (at 29.21 45.72 0)
@@
     (pin "6")
   )
-  (symbol (lib_id "power:GND") (at 25.4 60.96 0)
-    (in_bom yes) (on_board yes)
-    (property "Reference" "#PWR0402" (id 0) (at 25.4 67.31 0)
+  (symbol (lib_id "power:GND") (at 25.4 60.96 0) (unit 1)
+    (in_bom yes) (on_board yes)
+    (property "Reference" "#PWR0601" (id 0) (at 25.4 67.31 0)
       (effects (font (size 1.27 1.27)) hide)
     )
@@
   (symbol (lib_id "Device:R") (at 115.57 101.6 90) (unit 1)
     (in_bom yes) (on_board yes)
-    (property "Reference" "R401" (id 0) (at 115.57 96.3422 90))
+    (property "Reference" "R601" (id 0) (at 115.57 96.3422 90))
     (property "Value" "10k" (id 1) (at 115.57 98.6536 90))
     (property "Footprint" "Resistor_SMD:R_0402_1005Metric" (id 2) (at 115.57 103.378 90)
@@
   (symbol (lib_id "Device:R") (at 115.57 120.65 90) (unit 1)
     (in_bom yes) (on_board yes)
-    (property "Reference" "R402" (id 0) (at 115.57 115.3922 90))
+    (property "Reference" "R602" (id 0) (at 115.57 115.3922 90))
     (property "Value" "10k" (id 1) (at 115.57 117.7036 90))
     (property "Footprint" "Resistor_SMD:R_0402_1005Metric" (id 2) (at 115.57 122.428 90)
@@
   (symbol (lib_id "Interface_USB:CH340C") (at 52.07 127 0) (unit 1)
     (in_bom yes) (on_board yes)
-    (property "Reference" "U401" (id 0) (at 53.34 109.22 0)
+    (property "Reference" "U601" (id 0) (at 53.34 109.22 0)
       (effects (font (size 1.27 1.27)) (justify left))
     )
@@
   (symbol (lib_id "SH-ESP32:S8050") (at 130.81 101.6 0) (unit 1)
     (in_bom yes) (on_board yes)
-    (property "Reference" "Q401" (id 0) (at 135.636 100.4316 0)
+    (property "Reference" "Q601" (id 0) (at 135.636 100.4316 0)
       (effects (font (size 1.27 1.27)) (justify left))
     )
@@
   (symbol (lib_id "SH-ESP32:S8050") (at 130.81 120.65 0) (mirror x) (unit 1)
     (in_bom yes) (on_board yes)
-    (property "Reference" "Q402" (id 0) (at 135.636 119.4816 0)
+    (property "Reference" "Q602" (id 0) (at 135.636 119.4816 0)
       (effects (font (size 1.27 1.27)) (justify left))
     )
@@
   (symbol (lib_id "Device:C") (at 177.8 43.18 0) (unit 1)
     (in_bom yes) (on_board yes)
-    (property "Reference" "C402" (id 0) (at 180.721 42.0116 0)
+    (property "Reference" "C604" (id 0) (at 180.721 42.0116 0)
       (effects (font (size 1.27 1.27)) (justify left))
     )
@@
     (pin "2")
   )
-  (symbol (lib_id "power:GND") (at 177.8 46.99 0)
-    (in_bom yes) (on_board yes)
-    (property "Reference" "#PWR0405" (id 0) (at 177.8 53.34 0)
+  (symbol (lib_id "power:GND") (at 177.8 46.99 0) (unit 1)
+    (in_bom yes) (on_board yes)
+    (property "Reference" "#PWR0608" (id 0) (at 177.8 53.34 0)
       (effects (font (size 1.27 1.27)) hide)
     )
@@
     (pin "1")
   )
-  (symbol (lib_id "power:GND") (at 52.07 142.24 0)
-    (in_bom yes) (on_board yes)
-    (property "Reference" "#PWR0404" (id 0) (at 52.07 148.59 0)
+  (symbol (lib_id "power:GND") (at 52.07 142.24 0) (unit 1)
+    (in_bom yes) (on_board yes)
+    (property "Reference" "#PWR0602" (id 0) (at 52.07 148.59 0)
       (effects (font (size 1.27 1.27)) hide)
     )
@@
     (pin "1")
   )
-  (symbol (lib_id "power:GND") (at 91.44 71.12 0)
-    (in_bom yes) (on_board yes)
-    (property "Reference" "#PWR0406" (id 0) (at 91.44 77.47 0)
+  (symbol (lib_id "power:GND") (at 91.44 71.12 0) (unit 1)
+    (in_bom yes) (on_board yes)
+    (property "Reference" "#PWR0605" (id 0) (at 91.44 77.47 0)
       (effects (font (size 1.27 1.27)) hide)
     )
@@
   (symbol (lib_id "SH-ESP32:RCLAMP0524P-N") (at 92.71 57.15 0) (unit 1)
     (in_bom yes) (on_board yes)
-    (property "Reference" "U402" (id 0) (at 92.71 46.355 0))
+    (property "Reference" "U602" (id 0) (at 92.71 46.355 0))
     (property "Value" "RCLAMP0524P-N" (id 1) (at 92.71 48.6664 0))
     (property "Footprint" "Package_DFN_QFN:Diodes_UDFN-10_1.0x2.5mm_P0.5mm" (id 2) (at 92.71 59.69 0)
@@
     (pin "9")
   )
-  (symbol (lib_id "Device:Ferrite_Bead") (at 67.31 39.37 270) (unit 1)
-    (in_bom yes) (on_board yes)
-    (property "Reference" "FB401" (id 0) (at 67.31 32.4104 90))
+  (symbol (lib_id "Device:FerriteBead") (at 67.31 39.37 270) (unit 1)
+    (in_bom yes) (on_board yes)
+    (property "Reference" "FB601" (id 0) (at 67.31 32.4104 90))
     (property "Value" "GZ2012D601TF" (id 1) (at 67.31 34.7218 90))
     (property "Footprint" "Inductor_SMD:L_0805_2012Metric" (id 2) (at 67.31 37.592 90)
@@
   (symbol (lib_id "Device:C") (at 114.3 52.07 0) (unit 1)
     (in_bom yes) (on_board yes)
-    (property "Reference" "C403" (id 0) (at 117.221 50.9016 0)
+    (property "Reference" "C602" (id 0) (at 117.221 50.9016 0)
       (effects (font (size 1.27 1.27)) (justify left))
     )
@@
   (symbol (lib_id "Device:C") (at 127 49.53 0) (unit 1)
     (in_bom yes) (on_board yes)
-    (property "Reference" "C404" (id 0) (at 129.921 48.3616 0)
+    (property "Reference" "C603" (id 0) (at 129.921 48.3616 0)
       (effects (font (size 1.27 1.27)) (justify left))
     )
@@
     (pin "2")
   )
-  (symbol (lib_id "power:GND") (at 114.3 57.15 0)
-    (in_bom yes) (on_board yes)
-    (property "Reference" "#PWR0407" (id 0) (at 114.3 63.5 0)
+  (symbol (lib_id "power:GND") (at 114.3 57.15 0) (unit 1)
+    (in_bom yes) (on_board yes)
+    (property "Reference" "#PWR0606" (id 0) (at 114.3 63.5 0)
       (effects (font (size 1.27 1.27)) hide)
     )
@@
     (pin "1")
   )
-  (symbol (lib_id "power:GND") (at 127 57.15 0)
-    (in_bom yes) (on_board yes)
-    (property "Reference" "#PWR0408" (id 0) (at 127 63.5 0)
+  (symbol (lib_id "power:GND") (at 127 57.15 0) (unit 1)
+    (in_bom yes) (on_board yes)
+    (property "Reference" "#PWR0607" (id 0) (at 127 63.5 0)
       (effects (font (size 1.27 1.27)) hide)
     )
@@
     (pin "1")
   )
-  (symbol (lib_id "Device:Fuse") (at 48.26 39.37 270)
-    (in_bom yes) (on_board yes)
-    (property "Reference" "F401" (id 0) (at 48.26 34.3662 90))
+  (symbol (lib_id "Device:Fuse") (at 48.26 39.37 270) (unit 1)
+    (in_bom yes) (on_board yes)
+    (property "Reference" "F601" (id 0) (at 48.26 34.3662 90))
     (property "Value" "ASMD1206-050" (id 1) (at 48.26 36.6776 90))
     (property "Footprint" "Fuse:Fuse_1206_3216Metric" (id 2) (at 48.26 37.592 90)
@@
   (symbol (lib_id "power:+3.3V") (at 69.85 95.25 0) (unit 1)
     (in_bom yes) (on_board yes)
-    (property "Reference" "#PWR0109" (id 0) (at 69.85 99.06 0)
+    (property "Reference" "#PWR0604" (id 0) (at 69.85 99.06 0)
       (effects (font (size 1.27 1.27)) hide)
     )
@@
   (symbol (lib_id "Device:C") (at 59.69 54.61 0) (unit 1)
     (in_bom yes) (on_board yes)
-    (property "Reference" "C503" (id 0) (at 62.611 53.4416 0)
+    (property "Reference" "C601" (id 0) (at 62.611 53.4416 0)
       (effects (font (size 1.27 1.27)) (justify left))
     )
@@
     (pin "2")
   )
-  (symbol (lib_id "power:GND") (at 59.69 60.96 0)
-    (in_bom yes) (on_board yes)
-    (property "Reference" "#PWR0506" (id 0) (at 59.69 67.31 0)
-      (effects (font (size 1.27 1.27)) hide)
-    )
+  (symbol (lib_id "power:GND") (at 59.69 60.96 0) (unit 1)
+    (in_bom yes) (on_board yes)
+    (property "Reference" "#PWR0603" (id 0) (at 59.69 67.31 0)
+      (effects (font (size 1.27 1.27)) hide)
+    )
