File: I2C.kicad_sch (KiCad schematic)
At the start: 14 parts, among them J701 Conn_01x04, J702 Conn_01x04, U701 RCLAMP0524P-N

Commit message: Rename and update layout
Parts:
- removed C701: 10uF, Capacitor_SMD:C_0402_1005Metric, symbol Device:C
- removed C702, C703: 33pF, Capacitor_SMD:C_0402_1005Metric, symbol Device:C
- removed C704: 10uF/50V, Capacitor_SMD:C_1206_3216Metric, symbol Device:C
- removed C705, C706: 33pF/50V, Capacitor_SMD:C_0603_1608Metric, symbol Device:C
- removed FB701: GZ2012D601TF, Inductor_SMD:L_0805_2012Metric, symbol Device:Ferrite_Bead
- removed FB702, FB703: GZ2012D101TF, Inductor_SMD:L_0805_2012Metric, symbol Device:Ferrite_Bead
- removed J701: Conn_01x04, Connector_JST:JST_SH_BM04B-SRSS-TB_1x04-1MP_P1.00mm_Vertical, symbol Connector_Generic:Conn_01x04
- removed R701, R702: 2k, Resistor_SMD:R_0402_1005Metric, symbol Device:R
- removed U701: RCLAMP0524P-N, Package_DFN_QFN:Diodes_UDFN-10_1.0x2.5mm_P0.5mm, symbol SH-ESP32:RCLAMP0524P-N
- renumbered J702 to J501
Connections:
- net SCL_CONN is gone; now on net SCL: J501.3 (Pin_3)
- net SDA_CONN is gone; now on net SDA: J501.4 (Pin_4)
- net GND renamed GND1
- net I2C_3V3 renamed +3V3_1
- no-connect marks 2 -> 0
Other:
- note removed: "I2C (qwiic)"
- title: Sailor Hat with ESP32 -> SH-wg
- moved on the sheet: J501

Commit message: Finish 0.1.0 design
Other:
- title: SH-wg -> Sailor Hat WiFi Gateway
Changed lines of the file:
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@@
   (paper "A4")
   (title_block
-    (title "SH-wg")
+    (title "Sailor Hat WiFi Gateway")
     (date "2022-01-25")
     (rev "0.1.0")
@@
     (pin "4")
   )
-  (symbol (lib_id "SH-ESP32-mini:+3V3_1") (at 93.98 82.55 0) (unit 1)
+  (symbol (lib_id "SH-wg:+3V3_1") (at 93.98 82.55 0) (unit 1)
     (in_bom yes) (on_board yes) (fields_autoplaced)
     (property "Reference" "#PWR0502" (id 0) (at 93.98 86.36 0)
