File: canbus.kicad_sch (KiCad schematic)
At the start: 19 parts, among them J501 Conn_01x02, J601 Conn_01x04, U501 SN65HVD231, U502 ADuM1201AR, U603 PJ75AL33SA

Commit message: Rename and update layout
Parts:
- removed C504, C604: 100nF, Capacitor_SMD:C_0402_1005Metric, symbol Device:C
- removed C601: 10nF/50V, Capacitor_SMD:C_0402_1005Metric, symbol Device:C
- removed C603: 10uF/50V, Capacitor_SMD:C_1206_3216Metric, symbol Device:C
- removed C605: 10uF/10V, Capacitor_SMD:C_0603_1608Metric, symbol Device:C
- removed D601: SMBJ33CA, Diode_SMD:D_SMB, symbol Device:D_TVS
- removed D602: B5819W, Diode_SMD:D_SOD-123, symbol Device:D_Schottky
- removed F601: mSMD050-60V, Fuse:Fuse_1812_4532Metric, symbol Device:Polyfuse
- removed FB601: GZ2012D601TF, Inductor_SMD:L_0805_2012Metric, symbol Device:Ferrite_Bead
- removed J501: Conn_01x02, Connector_PinHeader_2.54mm:PinHeader_1x02_P2.54mm_Vertical, symbol Connector_Generic:Conn_01x02
- removed JP601: SolderJumper_2_Open, SH-ESP32:SolderJumper-2_P1.3mm_Open_TrianglePad_Narrow, symbol Jumper:SolderJumper_2_Open
- removed R601, R602: 240R, Resistor_SMD:R_0805_2012Metric, symbol Device:R
- removed U502: ADuM1201AR, Package_SO:SOIC-8_3.9x4.9mm_P1.27mm, symbol Isolator:ADuM1201AR
- removed U603: PJ75AL33SA, Package_TO_SOT_SMD:SOT-23, symbol SH-ESP32:HT75xx-1-SOT23
- added D201, D202: SMF24CA, Diode_SMD:D_SOD-123F, symbol Device:D_TVS
- J201: renamed from J601; value Conn_01x04 -> Conn_01x05; footprint Connector_Phoenix_MC:PhoenixContact_MCV_1,5_4-G-3.81_1x04_P3.81mm_Vertical -> SH-ESP32:M12-5A_Male_Horizontal_PCB_Hysik; symbol Connector_Generic:Conn_01x04 -> Connector_Generic:Conn_01x05; LCSC C8410 -> (none)
- renumbered C602 to C201, R503 to R201, U501 to U201
Connections:
- net D is gone; now on net CAN_TX: U201.1 (D)
- net R is gone; now on net CAN_RX: U201.4 (R)
- net CAN_H: now also J201.4 (Pin_4), D201.1 (A1); no longer J201.3 (Pin_3)
- net CAN_L: now also J201.5 (Pin_5), D202.2 (A2); no longer J201.4 (Pin_4)
- net CAN_3V3 renamed +3V3_1
- net CAN_GND renamed GND1
- net GND1: now also J201.3 (Pin_3), D201.2 (A2), D202.1 (A1); no longer J201.1 (Pin_1)
- no-connect marks 1 -> 2
Other:
- note removed: "5V power feed for the bus side of the CAN bus tranceiver"
- note removed: "Input voltage up to 35V. Output current at least 100mA."
- note removed: "Optional termination resistance for the bus"
- note removed: "WIRE-LINK from CAN12V_Prot to Vin_Prot"
- title: Sailor Hat with ESP32 -> SH-wg
- moved on the sheet: C201

Commit message: Finish 0.1.0 design
Other:
- title: SH-wg -> Sailor Hat WiFi Gateway
Changed lines of the file:
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@@
   (paper "A4")
   (title_block
-    (title "SH-wg")
+    (title "Sailor Hat WiFi Gateway")
     (date "2022-01-25")
     (rev "0.1.0")
@@
     (pin "1")
   )
-  (symbol (lib_id "SH-ESP32-mini:+3V3_1") (at 134.62 80.01 0) (unit 1)
+  (symbol (lib_id "SH-wg:+3V3_1") (at 134.62 80.01 0) (unit 1)
     (in_bom yes) (on_board yes) (fields_autoplaced)
     (property "Reference" "#PWR0205" (id 0) (at 134.62 83.82 0)

Commit message: Prepare final 0.1.0 proto
Parts:
- U201: value SN65HVD231 -> SN65HVD232DR; LCSC C129257 -> C30530
Changed lines of the file:
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@@
     (in_bom yes) (on_board yes)
     (property "Reference" "U201" (id 0) (at 137.16 100.33 0))
-    (property "Value" "SN65HVD231" (id 1) (at 142.24 102.87 0))
+    (property "Value" "SN65HVD232DR" (id 1) (at 142.24 102.87 0))
     (property "Footprint" "Package_SO:SOIC-8_3.9x4.9mm_P1.27mm" (id 2) (at 134.62 123.19 0)
       (effects (font (size 1.27 1.27)) hide)
@@
       (effects (font (size 1.27 1.27)) hide)
     )
-    (property "LCSC" " C129257" (id 4) (at 134.62 110.49 0)
+    (property "LCSC" "C30530" (id 4) (at 134.62 110.49 0)
       (effects (font (size 1.27 1.27)) hide)
     )

Commit message: Add a pull-up resistor to CAN TX line
Parts:
- added R202: 10k, Resistor_SMD:R_0402_1005Metric, symbol Device:R_Small
Connections:
- net +3V3_1: now also R202.1
- net CAN_TX: now also R202.2
Changed lines of the file:
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@@
   (junction (at 134.62 83.82) (diameter 0) (color 0 0 0 0)
+  )
+  (junction (at 160.02 107.95) (diameter 0) (color 0 0 0 0)
   )
   (no_connect (at 144.78 113.03))
@@
     (stroke (width 0) (type default) (color 0 0 0 0))
   )
+  (wire (pts (xy 160.02 107.95) (xy 168.91 107.95))
+    (stroke (width 0) (type default) (color 0 0 0 0))
+  )
   (wire (pts (xy 34.29 71.12) (xy 44.45 71.12))
     (stroke (width 0) (type default) (color 0 0 0 0))
@@
     (stroke (width 0) (type default) (color 0 0 0 0))
   )
-  (wire (pts (xy 144.78 107.95) (xy 151.13 107.95))
-    (stroke (width 0) (type default) (color 0 0 0 0))
-  )
   (wire (pts (xy 147.32 115.57) (xy 144.78 115.57))
     (stroke (width 0) (type default) (color 0 0 0 0))
@@
     (stroke (width 0) (type default) (color 0 0 0 0))
   )
+  (wire (pts (xy 144.78 107.95) (xy 160.02 107.95))
+    (stroke (width 0) (type default) (color 0 0 0 0))
+  )
   (wire (pts (xy 105.41 110.49) (xy 105.41 116.84))
     (stroke (width 0) (type default) (color 0 0 0 0))
@@
     (stroke (width 0) (type default) (color 0 0 0 0))
   )
+  (wire (pts (xy 160.02 105.41) (xy 160.02 107.95))
+    (stroke (width 0) (type default) (color 0 0 0 0))
+  )
   (wire (pts (xy 105.41 110.49) (xy 124.46 110.49))
     (stroke (width 0) (type default) (color 0 0 0 0))
@@
     (stroke (width 0) (type default) (color 0 0 0 0))
   )
+  (wire (pts (xy 160.02 97.79) (xy 160.02 100.33))
+    (stroke (width 0) (type default) (color 0 0 0 0))
+  )
   (wire (pts (xy 134.62 83.82) (xy 134.62 102.87))
     (stroke (width 0) (type default) (color 0 0 0 0))
@@
     (stroke (width 0) (type default) (color 0 0 0 0))
   )
-  (wire (pts (xy 144.78 110.49) (xy 151.13 110.49))
+  (wire (pts (xy 144.78 110.49) (xy 168.91 110.49))
     (stroke (width 0) (type default) (color 0 0 0 0))
   )
@@
     (effects (font (size 1.27 1.27)) (justify left))
   )
-  (hierarchical_label "CAN_TX" (shape input) (at 151.13 107.95 0)
+  (hierarchical_label "CAN_TX" (shape input) (at 168.91 107.95 0)
     (effects (font (size 1.27 1.27)) (justify left))
   )
-  (hierarchical_label "CAN_RX" (shape output) (at 151.13 110.49 0)
+  (hierarchical_label "CAN_RX" (shape output) (at 168.91 110.49 0)
     (effects (font (size 1.27 1.27)) (justify left))
   )
@@
       (effects (font (size 1.27 1.27)) hide)
     )
+    (pin "1")
+    (pin "2")
+  )
+  (symbol (lib_id "SH-wg:+3V3_1") (at 160.02 97.79 0) (unit 1)
+    (in_bom yes) (on_board yes) (fields_autoplaced)
+    (property "Reference" "#PWR0208" (id 0) (at 160.02 101.6 0)
+      (effects (font (size 1.27 1.27)) hide)
+    )
+    (property "Value" "+3V3_1" (id 1) (at 160.02 92.71 0))
+    (property "Footprint" "" (id 2) (at 160.02 97.79 0)
+      (effects (font (size 1.27 1.27)) hide)
+    )
+    (property "Datasheet" "" (id 3) (at 160.02 97.79 0)
+      (effects (font (size 1.27 1.27)) hide)
+    )
+    (pin "1")
+  )
+  (symbol (lib_id "Device:R_Small") (at 160.02 102.87 0) (unit 1)
+    (in_bom yes) (on_board yes)
+    (property "Reference" "R202" (id 0) (at 161.5186 101.7016 0)
+      (effects (font (size 1.27 1.27)) (justify left))
+    )
+    (property "Value" "10k" (id 1) (at 161.5186 104.013 0)
+      (effects (font (size 1.27 1.27)) (justify left))
+    )
+    (property "Footprint" "Resistor_SMD:R_0402_1005Metric" (id 2) (at 160.02 102.87 0)
+      (effects (font (size 1.27 1.27)) hide)
+    )
+    (property "Datasheet" "~" (id 3) (at 160.02 102.87 0)
+      (effects (font (size 1.27 1.27)) hide)
+    )
+    (property "LCSC" "C25744" (id 4) (at 160.02 102.87 0)
+      (effects (font (size 1.27 1.27)) hide)
+    )

Commit message: Update the design based on the test results
Other:
- note added: "Rs provides slope control to limit EMI on HVD230 and 231."
- note removed: "Rs provides slope control to limit EMI."
Changed lines of the file:
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@@
     (stroke (width 0) (type default) (color 0 0 0 0))
   )
-  (text "Rs provides slope control\nto limit EMI." (at 144.78 135.89 0)
+  (text "Rs provides slope control\nto limit EMI on HVD230\nand 231."
+    (at 152.4 129.54 0)
     (effects (font (size 1.27 1.27)) (justify left bottom))
   )
