File: SH-wg.kicad_sch (KiCad schematic)
At the start: 2 parts, among them J101 Aux PCB Conn Male, J102 Aux PCB Conn Female

Commit message: Add headers & LEDs
Other:
- sheet ESP32 ports: added CAN_LED_EN, RED_LED; removed none
- sheet User Interface ports: added CAN_LED_EN, CAN_RX, CAN_TX, RED_LED; removed none
- note added: "TODO: pins 1-6 should match the ESP-PROG programming header pin ordering!"

Commit message: Finish 0.1.0 design
Parts:
- J101: LCSC (none) -> C124388
- J102: LCSC (none) -> C36191
Other:
- sheet ESP32 ports: added ESP_RXD, ESP_TXD, HALL; removed RXD, TXD
- sheet User Interface ports: added HALL; removed HALL_OUTPUT
- note removed: "TODO: pins 1-6 should match the ESP-PROG programming header pin ordering!"
- title: SH-wg -> Sailor Hat WiFi Gateway
