File: SH-wg.kicad_pcb (KiCad board)
At the start: 4 copper layers, 54.6 x 99.2 mm, 85 parts, among them J101 Aux PCB Conn Male, J102 Aux PCB Conn Female, J201 Conn_01x05, J301 JTAG, J302 Digital IO, J303 Analog IO, J401 Power, J501 Conn_01x04, J701 Conn_02x03_Odd_Even, Q801 2N7002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

Commit message: Chore: C301 value: 1uf -> 1uF
Parts:
- C301: value 1uf -> 1uF
Changed lines of the file:
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@@
       (effects (font (size 1 1) (thickness 0.15)))
     )
-    (fp_text value "1uf" (at 0 1.17) (layer "F.Fab") hide
+    (fp_text value "1uF" (at 0 1.17) (layer "F.Fab") hide
       (effects (font (size 1 1) (thickness 0.15)))
     )
