File: SH-wg.kicad_pcb (KiCad board)
At the start: 4 copper layers, 54.6 x 99.2 mm, 85 parts, among them J101 Aux PCB Conn Male, J102 Aux PCB Conn Female, J201 Conn_01x05, J301 JTAG, J302 Digital IO, J303 Analog IO, J401 Power, J501 Conn_01x04, J701 Conn_02x03_Odd_Even, Q801 2N7002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

Commit message: Adjust tab locations
Parts:
- moved REF** 3.38 mm to (77.6, 82.7)
- moved REF** 3.30 mm to (42.2, 60.9)
- moved REF** 0.31 mm to (77.6, 39.1)
Changed lines of the file:
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@@
   )
   (footprint "kikit:Tab" (layer "F.Cu")
-    (at 80.8 83.75 90)
+    (at 77.6 82.65 90)
     (descr "A symbol representing annotation for tab placement")
     (attr board_only exclude_from_pos_files exclude_from_bom)
@@
   )
   (footprint "kikit:Tab" (layer "F.Cu")
-    (at 77.285 39.12 -90)
+    (at 77.6 39.12 -90)
     (descr "A symbol representing annotation for tab placement")
     (attr board_only exclude_from_pos_files exclude_from_bom)
@@
   )
   (footprint "kikit:Tab" (layer "F.Cu")
-    (at 42.25 57.6)
+    (at 42.2 60.9)
     (descr "A symbol representing annotation for tab placement")
     (attr board_only exclude_from_pos_files exclude_from_bom)

Commit message: Change CAN transceiver according to availability
Parts:
- U201: value SN65HVD232DR -> SN65HVD231DR
Other:
- board text added: "SHLD"
- board text added: "v1.0.0"
- board text removed: "v0.2.0"
Changed lines of the file:
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@@
     (descr "SOIC, 8 Pin (JEDEC MS-012AA, https://www.analog.com/media/en/package-pcb-resources/package/pkg_pdf/soic_narrow-r/r_8.pdf), generated with kicad-footprint-generator ipc_gullwing_generator.py")
     (tags "SOIC SO")
-    (property "LCSC" "C30530")
+    (property "LCSC" "C129257")
     (property "Sheetfile" "canbus.kicad_sch")
     (property "Sheetname" "CAN bus")
@@
       (effects (font (size 1 1) (thickness 0.15)))
     )
-    (fp_text value "SN65HVD232DR" (at 0 3.4) (layer "F.Fab") hide
+    (fp_text value "SN65HVD231DR" (at 0 3.4) (layer "F.Fab") hide
       (effects (font (size 1 1) (thickness 0.15)))
     )
@@
     (effects (font (size 0.8 0.8) (thickness 0.15)) (justify mirror))
   )
+  (gr_text "SHLD" (at 87.9 124 180) (layer "B.SilkS")
+    (effects (font (size 0.8 0.8) (thickness 0.15)) (justify mirror))
+  )
   (gr_text "Sailor Hat\nWiFi Gateway" (at 64.685 123.72 -180) (layer "B.SilkS")
     (effects (font (size 1.8 1.6) (thickness 0.35)) (justify left mirror))
@@
     (effects (font (size 0.8 0.8) (thickness 0.15)) (justify mirror))
   )
-  (gr_text "v0.2.0" (at 67.685 119.62 180) (layer "B.SilkS")
+  (gr_text "v1.0.0" (at 67.685 119.62 180) (layer "B.SilkS")
     (effects (font (size 1.2 1.2) (thickness 0.25)) (justify mirror))
   )
@@
     (effects (font (size 1.2 1.2) (thickness 0.25)) (justify left))
   )
-  (gr_text "v0.2.0" (at 80.285 51.12) (layer "F.SilkS")
+  (gr_text "v1.0.0" (at 80.285 51.12) (layer "F.SilkS")
     (effects (font (size 1.2 1.2) (thickness 0.25)))
   )

Commit message: Tweak tab locations
Parts:
- moved REF** 0.15 mm to (42.0, 60.9)
- moved REF** 0.15 mm to (42.6, 127.5)
- moved REF** 0.14 mm to (96.7, 44.9)
- moved REF** 0.10 mm to (77.6, 82.8)
- moved REF** 0.10 mm to (97.3, 127.6)
- moved REF** 0.10 mm to (70.0, 138.9)
- moved REF** 0.10 mm to (70.0, 116.2)
- moved REF** 0.07 mm to (77.6, 39.0)
- moved REF** 0.06 mm to (96.6, 70.5)
Changed lines of the file:
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@@
   )
   (footprint "kikit:Tab" (layer "F.Cu")
-    (at 77.6 82.65 90)
+    (at 77.6 82.75 90)
     (descr "A symbol representing annotation for tab placement")
     (attr board_only exclude_from_pos_files exclude_from_bom)
@@
     )
   )
+  (footprint "kikit:Tab" (layer "F.Cu")
+    (at 96.65 44.9 180)
+    (descr "A symbol representing annotation for tab placement")
+    (attr board_only exclude_from_pos_files exclude_from_bom)
+    (fp_text reference "REF**" (at 0 -2) (layer "F.SilkS") hide
+      (effects (font (size 1 1) (thickness 0.15)))
+    )
+    (fp_text value "Tab" (at -2.75 -1) (layer "Dwgs.User") hide
+      (effects (font (size 1.2 1.2) (thickness 0.2)))
+    )
+    (fp_text user "KIKIT: width: 4mm" (at -5.5 0 90) (layer "Dwgs.User") hide
+      (effects (font (size 1 1) (thickness 0.15)))
+    )
+    (fp_line (start 0.25 0) (end -0.75 -1) (layer "Dwgs.User") (width 0.3))
+    (fp_line (start 0.25 0) (end -0.75 1) (layer "Dwgs.User") (width 0.3))
+    (fp_line (start 0.25 0) (end -2.75 0) (layer "Dwgs.User") (width 0.3))
+    (fp_line (start 0.25 1) (end 0.25 -1) (layer "Dwgs.User") (width 0.3))
+  )
   (footprint "Capacitor_SMD:C_0402_1005Metric" (layer "F.Cu")
     (at 51.5 134)
@@
   )
   (footprint "kikit:Tab" (layer "F.Cu")
-    (at 42.75 127.5)
+    (at 42.6 127.5)
     (descr "A symbol representing annotation for tab placement")
     (attr board_only exclude_from_pos_files exclude_from_bom)
@@
   )
   (footprint "kikit:Tab" (layer "F.Cu")
-    (at 97.25 127.62 180)
+    (at 97.35 127.62 180)
     (descr "A symbol representing annotation for tab placement")
     (attr board_only exclude_from_pos_files exclude_from_bom)
@@
   )
   (footprint "kikit:Tab" (layer "F.Cu")
-    (at 96.535 44.82 180)
-    (descr "A symbol representing annotation for tab placement")
-    (attr board_only exclude_from_pos_files exclude_from_bom)
-    (fp_text reference "REF**" (at 0 -2) (layer "F.SilkS") hide
-      (effects (font (size 1 1) (thickness 0.15)))
-    )
-    (fp_text value "Tab" (at -2.75 -1) (layer "Dwgs.User") hide
-      (effects (font (size 1.2 1.2) (thickness 0.2)))
-    )
-    (fp_text user "KIKIT: width: 4mm" (at -5.5 0 90) (layer "Dwgs.User") hide
-      (effects (font (size 1 1) (thickness 0.15)))
-    )
-    (fp_line (start 0.25 0) (end -0.75 -1) (layer "Dwgs.User") (width 0.3))
-    (fp_line (start 0.25 1) (end 0.25 -1) (layer "Dwgs.User") (width 0.3))
-    (fp_line (start 0.25 0) (end -0.75 1) (layer "Dwgs.User") (width 0.3))
-    (fp_line (start 0.25 0) (end -2.75 0) (layer "Dwgs.User") (width 0.3))
-  )
-  (footprint "kikit:Tab" (layer "F.Cu")
-    (at 70 138.85 90)
+    (at 70 138.95 90)
     (descr "A symbol representing annotation for tab placement")
     (attr board_only exclude_from_pos_files exclude_from_bom)
@@
   )
   (footprint "kikit:Tab" (layer "F.Cu")
-    (at 77.6 39.12 -90)
+    (at 77.6 39.05 -90)
     (descr "A symbol representing annotation for tab placement")
     (attr board_only exclude_from_pos_files exclude_from_bom)
@@
   )
   (footprint "kikit:Tab" (layer "F.Cu")
-    (at 42.2 60.9)
+    (at 42.05 60.9)
     (descr "A symbol representing annotation for tab placement")
     (attr board_only exclude_from_pos_files exclude_from_bom)
@@
   )
   (footprint "kikit:Tab" (layer "F.Cu")
-    (at 70 116.35 -90)
+    (at 70 116.25 -90)
     (descr "A symbol representing annotation for tab placement")
     (attr board_only exclude_from_pos_files exclude_from_bom)
@@
   )
   (footprint "kikit:Tab" (layer "F.Cu")
-    (at 96.535 70.52 180)
+    (at 96.6 70.52 180)
     (descr "A symbol representing annotation for tab placement")
     (attr board_only exclude_from_pos_files exclude_from_bom)
@@
       (effects (font (size 1 1) (thickness 0.15)))
     )
+    (fp_line (start 0.25 0) (end -2.75 0) (layer "Dwgs.User") (width 0.3))
+    (fp_line (start 0.25 0) (end -0.75 1) (layer "Dwgs.User") (width 0.3))
+    (fp_line (start 0.25 1) (end 0.25 -1) (layer "Dwgs.User") (width 0.3))
     (fp_line (start 0.25 0) (end -0.75 -1) (layer "Dwgs.User") (width 0.3))
-    (fp_line (start 0.25 0) (end -0.75 1) (layer "Dwgs.User") (width 0.3))
-    (fp_line (start 0.25 0) (end -2.75 0) (layer "Dwgs.User") (width 0.3))
-    (fp_line (start 0.25 1) (end 0.25 -1) (layer "Dwgs.User") (width 0.3))
   )
   (footprint "Connector_PinHeader_2.54mm:PinHeader_2x03_P2.54mm_Vertical" (layer "B.Cu")
